File: KiCad-Files/Stromzaehler-V2.kicad_pcb (KiCad board)
At the start: 4 copper layers, 28 x 28.7 mm, 37 parts, among them J1 USB_C_Receptacle_USB2.0, J2 IO, J4 TagConnect TX2030, J5 PWR, J6 Gas Counter, Q1 Q_Photo_NPN, Q2 PJC7400_R1_00001, U1 ESP32­PICO­MINI­02U, U2 SN74AUP2G17, U4 TLV62568DBV

Commit message: finished testing device
Parts:
- C5: value 22nF -> DNP; footprint Franz-Lib:C_0402_1005Metric_NoSilk -> Franz-Lib:C_0402_1005Metric_NoSilk_DNP
- D2: value LED -> 15400385A3590
- Q1: value Q_Photo_NPN -> 1540032NA3090
- R9: footprint Franz-Lib:R_0402_1005Metric_NoSilk -> Franz-Lib:R_0402_1005Metric_NoSilk_DNP
