File: KiCad-Files/Stromzaehler-V2.kicad_sch (KiCad schematic)
At the start: 35 parts, among them J1 USB_C_Receptacle_USB2.0, J2 IO, J4 TagConnect TX2030, J5 PWR, J6 Gas Counter, Q1 1540032NA3090, Q2 PJC7400_R1_00001, U1 ESP32­PICO­MINI­02U, U2 SN74AUP2G17, U4 TLV62568DBV

Commit message: finished testing device
Parts:
- C5: value 22nF -> DNP; footprint Franz-Lib:C_0402_1005Metric_NoSilk -> Franz-Lib:C_0402_1005Metric_NoSilk_DNP
- R9: footprint Franz-Lib:R_0402_1005Metric_NoSilk -> Franz-Lib:R_0402_1005Metric_NoSilk_DNP
Changed lines of the file:
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@@
       (effects (font (size 1.27 1.27)) (justify right))
     )
-    (property "Footprint" "Franz-Lib:R_0402_1005Metric_NoSilk" (id 2) (at 53.34 140.97 0)
+    (property "Footprint" "Franz-Lib:R_0402_1005Metric_NoSilk_DNP" (id 2) (at 53.34 140.97 0)
       (effects (font (size 1.27 1.27)) hide)
     )
@@
       (effects (font (size 1.27 1.27)) (justify left))
     )
-    (property "Value" "22nF" (id 1) (at 237.2741 145.2185 0)
-      (effects (font (size 1.27 1.27)) (justify left))
-    )
-    (property "Footprint" "Franz-Lib:C_0402_1005Metric_NoSilk" (id 2) (at 234.95 143.51 0)
+    (property "Value" "DNP" (id 1) (at 237.2741 145.2185 0)
+      (effects (font (size 1.27 1.27)) (justify left))
+    )
+    (property "Footprint" "Franz-Lib:C_0402_1005Metric_NoSilk_DNP" (id 2) (at 234.95 143.51 0)
       (effects (font (size 1.27 1.27)) hide)
     )
@@
     )
     (path "/d0a86c67-e1ab-456f-a619-e243aff167df"
-      (reference "C5") (unit 1) (value "22nF") (footprint "Franz-Lib:C_0402_1005Metric_NoSilk")
+      (reference "C5") (unit 1) (value "DNP") (footprint "Franz-Lib:C_0402_1005Metric_NoSilk_DNP")
     )
     (path "/d6cbff75-5c2b-4b47-9942-8467e7759074"
@@
     )
     (path "/29da2067-8a40-4b9d-b070-795b0f9e23a9"
-      (reference "R9") (unit 1) (value "DNP") (footprint "Franz-Lib:R_0402_1005Metric_NoSilk")
+      (reference "R9") (unit 1) (value "DNP") (footprint "Franz-Lib:R_0402_1005Metric_NoSilk_DNP")
     )
     (path "/a761d759-6c8c-4e8c-8f3a-5a11e22f114c"
